File: hardware/Breakout_104pin_EEC-V-Connector/eecv-breakout.kicad_pcb (KiCad board)
At the start: 4 copper layers, 140.8 x 53.7 mm, 12 parts, among them J1 EEC-V, J2 Conn_01x13, J3 Conn_01x13, J4 Conn_01x13, J5 Conn_01x13, J6 Conn_01x13, J7 Conn_01x13, J8 Conn_01x13, J9 Conn_01x13

Commit message: Convert
Parts:
- G?: footprint rusefi_lib:LOGO -> gerefi_lib:LOGO
- G?: footprint rusefi_lib:Off_Road_Disclaimer -> gerefi_lib:Off_Road_Disclaimer
- J1: footprint rusefi_lib:eecv -> gerefi_lib:eecv
Other:
- board text added: "gerefi.com Rev. 0.3"
- board text removed: "rusefi.com Rev. 0.3"
Changed lines of the file:
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@@
   (net 103 "Net-(J1-Pad40)")
   (net 104 "Net-(J1-Pad14)")
-  (footprint "rusefi_lib:LOGO" (layer "F.Cu")
+  (footprint "gerefi_lib:LOGO" (layer "F.Cu")
     (at 93.62 56.13)
     (attr through_hole)
@@
       ) (layer "F.SilkS") (width 0.00254) (fill solid))
   )
-  (footprint "rusefi_lib:eecv" (layer "F.Cu")
+  (footprint "gerefi_lib:eecv" (layer "F.Cu")
     (at 93.62 20.36)
     (attr through_hole)
@@
     )
   )
-  (footprint "rusefi_lib:Off_Road_Disclaimer" (layer "F.Cu")
+  (footprint "gerefi_lib:Off_Road_Disclaimer" (layer "F.Cu")
     (at 28.85 53.59 90)
     (attr through_hole)
@@
     (effects (font (size 1 1) (thickness 0.15)))
   )
-  (gr_text "rusefi.com    Rev. 0.3" (at 159.406 54.352 -90) (layer "F.SilkS")
+  (gr_text "gerefi.com    Rev. 0.3" (at 159.406 54.352 -90) (layer "F.SilkS")
     (effects (font (size 1 1) (thickness 0.15)))
   )
