File: hardware/Breakout_112pin_Connector/Breakout_112pin_Connector.kicad_pcb (KiCad board)
At the start: 2 copper layers, 174 x 58 mm, 42 parts, among them J1 0643330100, J10 Conn_01x06, J11 Conn_01x06, J12 Conn_01x06, J13 Conn_01x06, J14 Conn_01x04, J15 Conn_01x04, J16 Conn_01x06, J17 Conn_01x06, J18 Conn_01x06, J19 Conn_01x06, J2 Conn_01x04, J20 Conn_01x04, J21 Conn_01x04, J22 Conn_01x06, J23 Conn_01x06, J24 Conn_01x06, J25 Conn_01x06, J26 Conn_01x01, J27 Conn_01x01, J28 Conn_01x04, J29 Conn_01x04, J3 Conn_01x04, J30 Conn_01x10, J31 Conn_01x10, J32 Conn_01x10, J33 Conn_01x10, J34 Conn_01x04, J35 Conn_01x04, J36 Conn_01x10, J37 Conn_01x10, J38 Conn_01x10, J39 Conn_01x10, J4 Conn_01x06, J5 Conn_01x06, J6 Conn_01x06, J7 Conn_01x06, J8 Conn_01x04, J9 Conn_01x04

Commit message: Convert
Parts:
- G? (x2): footprint rusefi:LOGO -> gerefi:LOGO
- G?: footprint rusefi:Off_Road_Disclaimer -> gerefi:Off_Road_Disclaimer
- J1: footprint rusefi_lib_private:64333-0100_1 -> gerefi_lib_private:64333-0100_1
Other:
- board text added: "gerEFI.com"
- board text removed: "rusEFI.com"
Changed lines of the file:
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@@
     (add_net "Net-(J1-PadH4)")
   )
-  (module rusefi:LOGO (layer B.Cu)
+  (module gerefi:LOGO (layer B.Cu)
     (at 243 73.5 180)
     (fp_text reference G? (at 0 -4.14782) (layer B.SilkS) hide
@@
       (xy 3.3528 0.39624)) (layer B.SilkS) (width 0.00254))
   )
-  (module rusefi:LOGO (layer F.Cu)
+  (module gerefi:LOGO (layer F.Cu)
     (at 243 73.5)
     (fp_text reference G? (at 0 4.14782) (layer F.SilkS) hide
@@
       (xy 3.3528 -0.39624)) (layer F.SilkS) (width 0.00254))
   )
-  (module rusefi:Off_Road_Disclaimer (layer B.Cu)
+  (module gerefi:Off_Road_Disclaimer (layer B.Cu)
     (at 167.75 69.5 180)
     (fp_text reference G? (at 0 5.715) (layer B.SilkS) hide
@@
     )
   )
-  (module rusefi_lib_private:64333-0100_1 (layer F.Cu)
+  (module gerefi_lib_private:64333-0100_1 (layer F.Cu)
     (at 167.915001 63.100001)
     (descr 64333-0100)
@@
     (pad MH4 thru_hole circle (at 58.05 23.85 180) (size 3.4 3.4) (drill 2.3) (layers *.Cu *.Mask)
       (net 1 Earth))
-    (model D:/GoogleDrive/MSDLab/KiCad/freelance/rusefi/rusefi_lib_private/643330100.stp
+    (model D:/GoogleDrive/MSDLab/KiCad/freelance/gerefi/gerefi_lib_private/643330100.stp
       (offset (xyz -4 0.5 2.5))
       (scale (xyz 1 1 1))
@@
     (effects (font (size 1 1) (thickness 0.15)))
   )
-  (gr_text rusEFI.com (at 243.25 78.25) (layer F.SilkS)
+  (gr_text gerEFI.com (at 243.25 78.25) (layer F.SilkS)
     (effects (font (size 1.5 1.5) (thickness 0.2)))
   )
-  (gr_text rusEFI.com (at 243.25 78.25) (layer B.SilkS)
+  (gr_text gerEFI.com (at 243.25 78.25) (layer B.SilkS)
     (effects (font (size 1.5 1.5) (thickness 0.2)) (justify mirror))
   )
