File: hardware/Breakout_112pin_Connector/Breakout_112pin_Connector.sch (KiCad schematic (older format))
At the start: 39 parts, among them J1 0643330100, J10 Conn_01x06, J11 Conn_01x06, J12 Conn_01x06, J13 Conn_01x06, J14 Conn_01x04, J15 Conn_01x04, J16 Conn_01x06, J17 Conn_01x06, J18 Conn_01x06, J19 Conn_01x06, J2 Conn_01x04, J20 Conn_01x04, J21 Conn_01x04, J22 Conn_01x06, J23 Conn_01x06, J24 Conn_01x06, J25 Conn_01x06, J26 Conn_01x01, J27 Conn_01x01, J28 Conn_01x04, J29 Conn_01x04, J3 Conn_01x04, J30 Conn_01x10, J31 Conn_01x10, J32 Conn_01x10, J33 Conn_01x10, J34 Conn_01x04, J35 Conn_01x04, J36 Conn_01x10, J37 Conn_01x10, J38 Conn_01x10, J39 Conn_01x10, J4 Conn_01x06, J5 Conn_01x06, J6 Conn_01x06, J7 Conn_01x06, J8 Conn_01x04, J9 Conn_01x04

Commit message: Convert
Parts:
- J1: footprint rusefi_lib_private:64333-0100_1 -> gerefi_lib_private:64333-0100_1
Changed lines of the file:
@@
 F 0 "J1" H 8175 9315 50  0000 C CNN
 F 1 "0643330100" H 8175 9224 50  0000 C CNN
-F 2 "rusefi_lib_private:64333-0100_1" H 8750 9200 50  0001 L CNN
+F 2 "gerefi_lib_private:64333-0100_1" H 8750 9200 50  0001 L CNN
 F 3 "https://www.molex.com/molex/products/part-detail/pcb_headers/0643330100" H 11350 7850 50  0001 L CNN
 F 4 "N/A" H 11350 7150 50  0001 L CNN "Mouser Part Number"
