File: hardware/Breakout_121pin_368255-2-Connector/368255-2.kicad_pcb (KiCad board)
At the start: 2 copper layers, 146.1 x 49.5 mm, 43 parts, among them P1 368255-2, P10 CONN_1, P11 CONN_1, P12 CONN_1, P13 CONN_1, P14 CONN_1, P15 CONN_1, P16 CONN_1, P17 CONN_1, P18 CONN_1, P19 CONN_1, P2 CONN_19, P20 CONN_1, P21 CONN_1, P22 CONN_1, P23 CONN_1, P24 CONN_1, P25 CONN_1, P26 CONN_1, P27 CONN_1, P28 CONN_1, P29 CONN_1, P3 CONN_19, P30 CONN_1, P31 CONN_1, P32 CONN_8, P33 CONN_8, P34 CONN_8, P35 CONN_8, P36 CONN_1, P37 CONN_1, P4 CONN_19, P5 CONN_19, P6 CONN_1, P7 CONN_1, P8 CONN_1, P9 CONN_1

Commit message: Convert
Parts:
- G?: footprint rusEFI_Lib:LOGO -> gerEFI_Lib:LOGO
- G?: footprint rusEFI_Lib:LOGO_F -> gerEFI_Lib:LOGO_F
- P1: footprint rusEFI_Lib:368255-2 -> gerEFI_Lib:368255-2
Other:
- board text added: "gerEFI.com R0.2"
- board text removed: "rusEFI.com R0.2"
Changed lines of the file:
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@@
     (pad 1 thru_hole circle (at 0 0) (size 4.064 4.064) (drill 3.048) (layers *.Cu *.Mask F.SilkS))
   )
-  (module rusEFI_Lib:LOGO (layer F.Cu)
+  (module gerEFI_Lib:LOGO (layer F.Cu)
     (at 194.945 92.075)
     (fp_text reference G? (at 0 4.14782) (layer F.SilkS) hide
@@
       (xy 3.3528 -0.39624) (xy 3.3528 -0.39624)) (layer F.SilkS) (width 0.00254))
   )
-  (module rusEFI_Lib:LOGO_F (layer B.Cu)
+  (module gerEFI_Lib:LOGO_F (layer B.Cu)
     (at 194.945 92.075)
     (fp_text reference G? (at 0 -4.14782) (layer B.SilkS) hide
@@
       (xy 3.3401 -0.50546) (xy 3.34264 -0.09398) (xy 3.34518 -0.04318) (xy 3.34518 -0.04318)) (layer B.SilkS) (width 0.00254))
   )
-  (module rusEFI_Lib:368255-2 (layer F.Cu)
+  (module gerEFI_Lib:368255-2 (layer F.Cu)
     (at 60.198 32.893)
     (fp_text reference P1 (at 138 68 270) (layer F.SilkS)
@@
     (effects (font (size 2 2) (thickness 0.25)))
   )
-  (gr_text "rusEFI.com  R0.2" (at 174.625 60.96) (layer B.SilkS)
+  (gr_text "gerEFI.com  R0.2" (at 174.625 60.96) (layer B.SilkS)
     (effects (font (size 2.032 1.524) (thickness 0.3048)) (justify mirror))
   )
-  (gr_text "rusEFI.com  R0.2" (at 174.879 60.579) (layer F.SilkS)
+  (gr_text "gerEFI.com  R0.2" (at 174.879 60.579) (layer F.SilkS)
     (effects (font (size 2.032 1.524) (thickness 0.3048)))
   )
