File: hardware/Breakout_134pin_7-967288-1-Connector/134pin_7-967288-1.kicad_pcb (KiCad board)
At the start: 2 copper layers, 139.7 x 73.7 mm, 40 parts, among them J1 Conn_01x03, J10 Conn_01x06, J11 Conn_01x06, J12 Conn_01x03, J13 Conn_01x03, J14 Conn_01x03, J15 Conn_01x13, J16 Conn_01x13, J17 Conn_01x13, J18 Conn_01x13, J19 Conn_01x13, J2 Conn_01x03, J20 Conn_01x13, J21 Conn_01x13, J22 Conn_01x13, J23 Conn_01x10, J24 Conn_01x10, J25 Conn_01x10, J26 Conn_01x10, J27 Conn_01x03, J28 Conn_01x03, J29 Conn_01x03, J3 Conn_01x03, J30 Conn_01x10, J31 Conn_01x10, J32 Conn_01x10, J33 Conn_01x10, J34 Conn_01x03, J35 Conn_01x03, J36 Conn_01x03, J37 Conn_01x01, J4 Conn_01x06, J5 Conn_01x06, J6 Conn_01x06, J7 Conn_01x06, J8 Conn_01x06, J9 Conn_01x06, P1 134pin_7-967288-1_KC5

Commit message: Convert
Parts:
- LOGO1: footprint rusEFI:LOGO -> gerEFI:LOGO
Other:
- board text added: "gerEFI.com 134pin 7-967288-1 R0.2"
- board text removed: "rusEFI.com 134pin 7-967288-1 R0.2"
Changed lines of the file:
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@@
     )
   )
-  (module rusEFI:LOGO (layer F.Cu)
+  (module gerEFI:LOGO (layer F.Cu)
     (at 210.82 97.79)
     (fp_text reference LOGO1 (at 0 4.14782) (layer F.SilkS) hide
@@
     (arrow2b (pts (xy 226.06 137.16) (xy 225.473579 136.033496)))
   )
-  (gr_text "rusEFI.com\n134pin 7-967288-1\nR0.2" (at 211.328 84.328 90) (layer F.SilkS)
+  (gr_text "gerEFI.com\n134pin 7-967288-1\nR0.2" (at 211.328 84.328 90) (layer F.SilkS)
     (effects (font (size 0.75 0.75) (thickness 0.13)))
   )
