File: hardware/Breakout_35pin_MX7-C-35PL-C11-connector/MX7-C-35PL-C11.kicad_pcb (KiCad board)
At the start: 2 copper layers, 47 x 35.6 mm, 13 parts, among them P1 CONN_1, P10 CONN_01X02, P11 CONN_01X08, P12 CONN_01X02, P13 CONN_01X02, P2 CONN_1, P3 CONN_01X02, P4 CONN_01X02, P5 CONN_01X07, P6 CONN_01X02, P7 CONN_01X04, P8 MX7-C-35PL-C11, P9 CONN_01X04

Commit message: Convert
Other:
- board text added: "gerEFI.com R0.2 MX7-C-35PL-C11"
- board text removed: "rusEFI.com R0.2 MX7-C-35PL-C11"
Changed lines of the file:
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@@
     (date 2017-03-30)
     (rev R0.2)
-    (company rusEFI)
+    (company gerEFI)
   )
   (layers
@@
     (effects (font (size 1.016 1.016) (thickness 0.127)) (justify mirror))
   )
-  (gr_text "rusEFI.com R0.2\nMX7-C-35PL-C11" (at 149.225 196.215) (layer B.SilkS)
+  (gr_text "gerEFI.com R0.2\nMX7-C-35PL-C11" (at 149.225 196.215) (layer B.SilkS)
     (effects (font (thickness 0.127)) (justify mirror))
   )
