File: hardware/Breakout_48pin_174917-Connector/174917.kicad_pcb (KiCad board)
At the start: 2 copper layers, 100 x 33.5 mm, 39 parts, among them P1 CONN_3, P10 CONN_1, P11 CONN_1, P12 CONN_1, P13 CONN_3, P14 CONN_3, P15 CONN_1, P16 CONN_1, P17 CONN_1, P18 CONN_1, P19 CONN_1, P2 CONN_3, P20 CONN_1, P21 CONN_1, P22 CONN_1, P23 CONN_1, P24 CONN_1, P25 174917, P26 CONN_8, P27 CONN_8, P3 CONN_1, P30 CONN_8, P31 CONN_8, P32 CONN_8, P33 CONN_8, P36 CONN_8, P37 CONN_8, P38 CONN_1, P39 CONN_1, P4 CONN_1, P40 CONN_1, P41 CONN_1, P5 CONN_1, P6 CONN_1, P7 CONN_1, P8 CONN_1, P9 CONN_1

Commit message: Convert
Other:
- board text added: "gerEFI by CrazyStriker Visit gerEFI.com"
- board text removed: "rusEFI by CrazyStriker Visit rusEFI.com"
Changed lines of the file:
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@@
     (arrow2b (pts (xy 212.089999 40.64) (xy 212.676419 41.766503)))
   )
-  (gr_text "rusEFI       by CrazyStriker\nVisit rusEFI.com" (at 60.5 72.5 90) (layer F.SilkS)
+  (gr_text "gerEFI       by CrazyStriker\nVisit gerEFI.com" (at 60.5 72.5 90) (layer F.SilkS)
     (effects (font (size 1.9 1.4) (thickness 0.3048)) (justify left))
   )
