File: hardware/Breakout_52pin_172319-1-Connector/172319-1_connector.kicad_pcb (KiCad board)
At the start: 2 copper layers, 124.5 x 33.7 mm, 3 parts, among them P1 172319-1, P2 172319-1, P3 CONN_01X01

Commit message: Convert
Parts:
- P1, P2: footprint rusEFI_Lib:172319-1_connector -> gerEFI_Lib:172319-1_connector
Other:
- board text added: "gerEFI.com R0.2"
- board text removed: "rusEFI.com R0.2"
Changed lines of the file:
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@@
     (date 2018-12-21)
     (rev R0.2)
-    (company "DAECU for rusEFI")
+    (company "DAECU for gerEFI")
   )
   (layers
@@
     (add_net "Net-(P1-Pad9)")
   )
-  (module rusEFI_Lib:172319-1_connector (layer F.Cu)
+  (module gerEFI_Lib:172319-1_connector (layer F.Cu)
     (at 71.12 108.585)
     (descr 172319-1_connector)
@@
     (pad 45 thru_hole circle (at 69.3 4.6 180) (size 1.89954 1.89954) (drill 1.50076) (layers *.Cu *.Mask F.SilkS)
       (net 53 "Net-(P1-Pad45)"))
-    (model ${KISYS3DMOD}../../../../../../Users/Vista_64_D630/Desktop/Jared/code/Hardware/trunk/rusefi.com/rusefi_lib/3d/c-172319-1-k3-3d.wrl
+    (model ${KISYS3DMOD}../../../../../../Users/Vista_64_D630/Desktop/Jared/code/Hardware/trunk/gerefi.com/gerefi_lib/3d/c-172319-1-k3-3d.wrl
       (at (xyz 2.015 1.18 0.43))
       (scale (xyz 1 1 1))
@@
     )
   )
-  (module rusEFI_Lib:172319-1_connector (layer B.Cu)
+  (module gerEFI_Lib:172319-1_connector (layer B.Cu)
     (at 71.12 121.92)
     (descr 172319-1_connector)
@@
     (pad 45 thru_hole circle (at 69.3 -4.6 180) (size 1.89954 1.89954) (drill 1.50076) (layers *.Cu *.Mask B.SilkS)
       (net 53 "Net-(P1-Pad45)"))
-    (model ${KISYS3DMOD}../../../../../../Users/Vista_64_D630/Desktop/Jared/code/Hardware/trunk/rusefi.com/rusefi_lib/3d/c-172319-1-k3-3d.wrl
+    (model ${KISYS3DMOD}../../../../../../Users/Vista_64_D630/Desktop/Jared/code/Hardware/trunk/gerefi.com/gerefi_lib/3d/c-172319-1-k3-3d.wrl
       (at (xyz 2.015 1.18 0.43))
       (scale (xyz 1 1 1))
@@
     (effects (font (size 2.032 1.524) (thickness 0.3048)) (justify mirror))
   )
-  (gr_text "rusEFI.com R0.2" (at 115.57 128.27) (layer B.SilkS)
+  (gr_text "gerEFI.com R0.2" (at 115.57 128.27) (layer B.SilkS)
     (effects (font (size 2.032 1.524) (thickness 0.3048)) (justify mirror))
   )
-  (gr_text "rusEFI.com R0.2" (at 115.57 128.524) (layer F.SilkS)
+  (gr_text "gerEFI.com R0.2" (at 115.57 128.524) (layer F.SilkS)
     (effects (font (size 2.032 1.524) (thickness 0.3048)))
   )
