File: hardware/Breakout_55pin-motronic-Connector/motronic-wire-adapter.kicad_pcb (KiCad board)
At the start: 2 copper layers, 157.5 x 48.5 mm, 10 parts, among them P1 MOTRONIC, P2 CONN_19, P3 CONN_18, P4 CONN_18, P5 CONN_1, P6 CONN_1

Commit message: Convert
Parts:
- P1: footprint rusEFI_Modules:55pin_china_bosch_motronic -> gerEFI_Modules:55pin_china_bosch_motronic
Other:
- board text added: "gerEfi 55 pin MOTRONIC 0.1"
- board text removed: "rusEfi 55 pin MOTRONIC 0.1"
Changed lines of the file:
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@@
     (add_net N-000009)
   )
-  (module rusEFI_Modules:55pin_china_bosch_motronic (layer F.Cu)
+  (module gerEFI_Modules:55pin_china_bosch_motronic (layer F.Cu)
     (at 220 168.5 180)
     (fp_text reference P1 (at 0 27.5) (layer F.SilkS) hide
@@
     (effects (font (size 1.5 2) (thickness 0.3)))
   )
-  (gr_text "rusEfi 55 pin\nMOTRONIC 0.1" (at 283 140.5 180) (layer F.SilkS)
+  (gr_text "gerEfi 55 pin\nMOTRONIC 0.1" (at 283 140.5 180) (layer F.SilkS)
     (effects (font (size 2 2) (thickness 0.3)))
   )
-  (gr_text "rusEfi 55 pin\nMOTRONIC 0.1" (at 282.448 140 180) (layer B.SilkS)
+  (gr_text "gerEfi 55 pin\nMOTRONIC 0.1" (at 282.448 140 180) (layer B.SilkS)
     (effects (font (size 2 2) (thickness 0.3)) (justify mirror))
   )
