File: hardware/Breakout_55pin_963063-15-Connector/963063-15.kicad_pcb (KiCad board)
At the start: 2 copper layers, 150 x 50 mm, 10 parts, among them P1 963063_15, P2 CONN_19, P3 CONN_18, P4 CONN_18, P5 CONN_1, P6 CONN_1

Commit message: Convert
Other:
- board text added: "gerEfi 55 pin TE 0.1"
- board text removed: "rusEfi 55 pin TE 0.1"
Changed lines of the file:
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@@
     (effects (font (size 1.5 2) (thickness 0.3)) (justify mirror))
   )
-  (gr_text "rusEfi 55 pin\nTE 0.1" (at 282.448 147.066 180) (layer F.SilkS)
+  (gr_text "gerEfi 55 pin\nTE 0.1" (at 282.448 147.066 180) (layer F.SilkS)
     (effects (font (size 2 2) (thickness 0.3)))
   )
-  (gr_text "rusEfi 55 pin\nTE 0.1" (at 282.448 147.066 180) (layer B.SilkS)
+  (gr_text "gerEfi 55 pin\nTE 0.1" (at 282.448 147.066 180) (layer B.SilkS)
     (effects (font (size 2 2) (thickness 0.3)) (justify mirror))
   )
