File: hardware/Breakout_60pin_EEC-IV-Connector/Breakout_60pin_EEC-IV.kicad_pcb (KiCad board)
At the start: 2 copper layers, 139.7 x 62.2 mm, 17 parts, among them J1 Conn_01x01, J10 Conn_01x10, J11 Conn_01x10, J12 Conn_01x10, J13 Conn_01x10, J14 EEC-IV, J2 Conn_01x10, J3 Conn_01x10, J4 Conn_01x10, J5 Conn_01x10, J6 Conn_01x10, J7 Conn_01x10, J8 Conn_01x10, J9 Conn_01x10

Commit message: Convert
Parts:
- G1: footprint rusEFI:Off_Road_Disclaimer -> gerEFI:Off_Road_Disclaimer
- G2: footprint rusEFI:LOGO -> gerEFI:LOGO
- J14: footprint rusEFI:eeciv -> gerEFI:eeciv
Other:
- board text added: "gerEFI.com R0.2"
- board text removed: "rusEFI.com R0.2"
Changed lines of the file:
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@@
     )
   )
-  (footprint "rusEFI:Off_Road_Disclaimer" (layer "F.Cu")
+  (footprint "gerEFI:Off_Road_Disclaimer" (layer "F.Cu")
     (at 165.1 104.14 90)
     (attr through_hole)
@@
     )
   )
-  (footprint "rusEFI:LOGO" (layer "F.Cu")
+  (footprint "gerEFI:LOGO" (layer "F.Cu")
     (at 111.2393 93.3704 90)
     (attr through_hole)
@@
     )
   )
-  (footprint "rusEFI:eeciv" (layer "F.Cu")
+  (footprint "gerEFI:eeciv" (layer "F.Cu")
     (at 166.009425 62.296099)
     (attr through_hole)
@@
     (effects (font (size 1.016 1.016) (thickness 0.13)))
   )
-  (gr_text "rusEFI.com  R0.2" (at 109.22 106.68 90) (layer "F.SilkS")
+  (gr_text "gerEFI.com  R0.2" (at 109.22 106.68 90) (layer "F.SilkS")
     (effects (font (size 1.016 1.016) (thickness 0.13)))
   )
