File: hardware/Breakout_64pin_176122-6-Connector/176122-6.kicad_pcb (KiCad board)
At the start: 2 copper layers, 137.2 x 41.5 mm, 28 parts, among them P1 CONN_3, P13 CONN_3, P14 CONN_3, P19 CONN_1, P2 CONN_3, P20 CONN_1, P25 0176122-06, P26 CONN_8, P27 CONN_8, P28 CONN_8, P29 CONN_8, P3 Conn_01x04_Male, P30 CONN_8, P31 CONN_8, P32 CONN_8, P33 CONN_8, P34 CONN_8, P35 CONN_8, P36 CONN_8, P37 CONN_8, P4 Conn_01x04_Male, P42 Conn_01x04_Male, P43 Conn_01x04_Male, P7 CONN_1, P8 CONN_1

Commit message: Convert
Parts:
- G1: footprint rusefi_lib:LOGO -> gerefi_lib:LOGO
Other:
- board text added: "gerEFI by DAECU gerEFI.com R0.3"
- board text removed: "rusEFI by DAECU rusEFI.com R0.3"
Changed lines of the file:
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@@
     )
   )
-  (module rusefi_lib:LOGO (layer F.Cu)
+  (module gerefi_lib:LOGO (layer F.Cu)
     (at 55.88 75.565 90)
     (fp_text reference G1 (at 0 4.14782 90) (layer F.SilkS) hide
@@
     )
   )
-  (gr_text "rusEFI by DAECU\nrusEFI.com\nR0.3" (at 56.515 51.435 90) (layer F.SilkS)
+  (gr_text "gerEFI by DAECU\ngerEFI.com\nR0.3" (at 56.515 51.435 90) (layer F.SilkS)
     (effects (font (size 2.032 1.524) (thickness 0.3048)))
   )
