File: hardware/Breakout_68pin_966595-1_and_963356-1-Connector/966595-1_and_963356-1.kicad_pcb (KiCad board)
At the start: 2 copper layers, 116 x 33 mm, 4 parts, among them P101 963356-1, P102 966595-1

Commit message: Convert
Parts:
- P101: footprint rusEFI_Lib:963356-1 -> gerEFI_Lib:963356-1
- P102: footprint rusEFI_Lib:966595-1 -> gerEFI_Lib:966595-1
Other:
- board text added: "gerEFI.com"
- board text removed: "rusEFI.com"
Changed lines of the file:
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@@
     (date 2017-12-16)
     (rev R0.1)
-    (company "DAECU for rusEFI")
+    (company "DAECU for gerEFI")
   )
   (layers
@@
     (add_net "Net-(P101-Pad9)")
   )
-  (module rusEFI_Lib:963356-1 (layer F.Cu)
+  (module gerEFI_Lib:963356-1 (layer F.Cu)
     (at 121 120)
     (descr 963356-1)
@@
     (pad 45 thru_hole circle (at 42 3.3 180) (size 1.49954 1.49954) (drill 1.10076) (layers *.Cu *.Mask F.SilkS)
       (net 69 "Net-(P101-Pad45)"))
-    (model ../../../../../../Users/Vista_64_D630/Desktop/Jared/code/Hardware/trunk/rusefi.com/rusefi_lib/3d/c-963356-1-d-3d.wrl
+    (model ../../../../../../Users/Vista_64_D630/Desktop/Jared/code/Hardware/trunk/gerefi.com/gerefi_lib/3d/c-963356-1-d-3d.wrl
       (at (xyz 0 -1.04 0.53))
       (scale (xyz 0.393701 0.393701 0.393701))
@@
     )
   )
-  (module rusEFI_Lib:966595-1 (layer B.Cu)
+  (module gerEFI_Lib:966595-1 (layer B.Cu)
     (at 121 100)
     (descr 966595-1)
@@
     (pad 45 thru_hole circle (at 42 0 180) (size 1.49954 1.49954) (drill 1.10076) (layers *.Cu *.Mask B.SilkS)
       (net 69 "Net-(P101-Pad45)"))
-    (model ../../../../../../Users/Vista_64_D630/Desktop/Jared/code/Hardware/trunk/rusefi.com/rusefi_lib/3d/c-966595-1-a1-3d.wrl
+    (model ../../../../../../Users/Vista_64_D630/Desktop/Jared/code/Hardware/trunk/gerefi.com/gerefi_lib/3d/c-966595-1-a1-3d.wrl
       (at (xyz 0 0 1.265))
       (scale (xyz 0.393701 0.393701 0.393701))
@@
     (arrow2b (pts (xy 184 94) (xy 184.586421 95.126504)))
   )
-  (gr_text rusEFI.com (at 70 106) (layer F.SilkS)
+  (gr_text gerEFI.com (at 70 106) (layer F.SilkS)
     (effects (font (size 2.032 1.524) (thickness 0.3048)))
   )
