File: hardware/Breakout_72pin_1123038-2-Connector/1123038-2.kicad_pcb (KiCad board)
At the start: 2 copper layers, 77.5 x 33.7 mm, 16 parts, among them P1 CONN_1, P10 1123038-2, P11 CONN_01X05, P12 CONN_01X05, P13 CONN_01X08, P14 CONN_01X06, P15 CONN_01X05, P2 CONN_1, P3 CONN_01X05, P4 CONN_01X06, P5 CONN_01X06, P6 CONN_01X05, P7 CONN_01X08, P8 CONN_01X08, P9 CONN_01X05

Commit message: Convert
Other:
- board text added: "gerEFI.com R0.3 1123038-2 connector break out"
- board text removed: "rusEFI.com R0.3 1123038-2 connector break out"
Changed lines of the file:
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@@
     (date 2017-03-19)
     (rev R0.4)
-    (company rusEFI)
+    (company gerEFI)
   )
   (layers
@@
     (effects (font (size 1.016 1.016) (thickness 0.127)) (justify mirror))
   )
-  (gr_text "rusEFI.com R0.3\n1123038-2 connector break out" (at 137.668 44.704) (layer B.SilkS)
+  (gr_text "gerEFI.com R0.3\n1123038-2 connector break out" (at 137.668 44.704) (layer B.SilkS)
     (effects (font (thickness 0.127)) (justify mirror))
   )
