File: hardware/Breakout_80pin_8-1393476-0/Breakout_80pin_1393476-Connector.kicad_pcb (KiCad board)
At the start: 2 copper layers, 144 x 58 mm, 24 parts, among them J1 8-1393476-0, J10 Conn_01x12, J11 Conn_01x14, J12 Conn_01x12, J13 Conn_01x14, J14 Conn_01x12, J15 Conn_01x12, J16 Conn_01x01, J17 Conn_01x01, J18 Conn_01x01, J19 Conn_01x01, J2 Conn_01x12, J20 Screw_Terminal_01x02, J21 Screw_Terminal_01x02, J3 Conn_01x12, J4 Conn_01x14, J5 Conn_01x12, J6 Screw_Terminal_01x02, J7 Conn_01x12, J8 Conn_01x14, J9 Screw_Terminal_01x02

Commit message: Convert
Parts:
- G?: footprint rusefi:Off_Road_Disclaimer -> gerefi:Off_Road_Disclaimer
- G? (x2): footprint rusefi:LOGO -> gerefi:LOGO
- J1: footprint rusefi:8-1393476-0 -> gerefi:8-1393476-0
Other:
- board text added: "gerEFI.com"
- board text removed: "rusEFI.com"
Changed lines of the file:
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@@
     (add_net "Net-(J1-Pad9)")
   )
-  (module rusefi:Off_Road_Disclaimer (layer B.Cu)
+  (module gerefi:Off_Road_Disclaimer (layer B.Cu)
     (at 159 62.5 180)
     (fp_text reference G? (at 0 5.715) (layer B.SilkS) hide
@@
     )
   )
-  (module rusefi:LOGO (layer F.Cu)
+  (module gerefi:LOGO (layer F.Cu)
     (at 39 94.5)
     (fp_text reference G? (at 0 4.14782) (layer F.SilkS) hide
@@
       (xy 3.3528 -0.39624)) (layer F.SilkS) (width 0.00254))
   )
-  (module rusefi:LOGO (layer B.Cu)
+  (module gerefi:LOGO (layer B.Cu)
     (at 39 94.5 180)
     (fp_text reference G? (at 0 -4.14782) (layer B.SilkS) hide
@@
       (net 79 "Net-(J1-Pad27)"))
   )
-  (module rusefi:8-1393476-0 (layer F.Cu)
+  (module gerefi:8-1393476-0 (layer F.Cu)
     (at 107 75 180)
     (fp_text reference J1 (at -69.100075 -7.810275) (layer F.SilkS)
@@
     (effects (font (size 1 1) (thickness 0.15)))
   )
-  (gr_text rusEFI.com (at 107 86) (layer B.SilkS)
+  (gr_text gerEFI.com (at 107 86) (layer B.SilkS)
     (effects (font (size 2 2) (thickness 0.25)) (justify mirror))
   )
   (gr_line (start 107 127) (end 107 50) (layer Dwgs.User) (width 0.15))
-  (gr_text rusEFI.com (at 107 86) (layer F.SilkS)
+  (gr_text gerEFI.com (at 107 86) (layer F.SilkS)
     (effects (font (size 2 2) (thickness 0.25)))
   )
