File: hardware/Breakout_80pin_8-1393476-0/Breakout_80pin_1393476-Connector.sch (KiCad schematic (older format))
At the start: 21 parts, among them J1 8-1393476-0, J10 Conn_01x12, J11 Conn_01x14, J12 Conn_01x12, J13 Conn_01x14, J14 Conn_01x12, J15 Conn_01x12, J16 Conn_01x01, J17 Conn_01x01, J18 Conn_01x01, J19 Conn_01x01, J2 Conn_01x12, J20 Screw_Terminal_01x02, J21 Screw_Terminal_01x02, J3 Conn_01x12, J4 Conn_01x14, J5 Conn_01x12, J6 Screw_Terminal_01x02, J7 Conn_01x12, J8 Conn_01x14, J9 Screw_Terminal_01x02

Commit message: Convert
Parts:
- J1: footprint rusefi:8-1393476-0 -> gerefi:8-1393476-0
Changed lines of the file:
@@
 F 0 "J1" H 6025 5617 50  0000 C CNN
 F 1 "8-1393476-0" H 6025 5526 50  0000 C CNN
-F 2 "rusefi:8-1393476-0" H 6025 3250 50  0001 L BNN
+F 2 "gerefi:8-1393476-0" H 6025 3250 50  0001 L BNN
 F 3 "MANUFACTURER RECOMMENDATIONS" H 6025 3250 50  0001 L BNN
 F 4 "TE CONNECTIVITY" H 6025 3250 50  0001 L BNN "Field4"
