File: hardware/Breakout_88pin_VAG-Connector/Bosch_88pin_Breakout.kicad_pcb (KiCad board)
At the start: 2 copper layers, 142 x 58 mm, 97 parts, among them J1 BOSCH_88PIN_02X44, J10 Pin17, J11 Pin19, J12 Pin21, J13 Pin23, J14 Pin25, J15 Pin27, J16 Pin29, J17 Pin31, J18 Pin33, J19 Pin35, J2 Pin1, J20 Pin37, J21 Pin39, J22 Pin41, J23 Pin43, J24 Pin45, J25 Pin47, J26 Pin49, J27 Pin51, J28 Pin53, J29 Pin55, J3 Pin3, J30 Pin57, J31 Pin59, J32 Pin61, J33 Pin63, J34 Pin65, J35 Pin67, J36 Pin69, J37 Pin71, J38 Pin73, J39 Pin75, J4 Pin5, J40 Pin77, J41 Pin79, J42 Pin81, J43 Pin83, J44 Pin85, J45 Pin87, J46 Pin2, J47 Pin4, J48 Pin6, J49 Pin8, J5 Pin7, J50 Pin10, J51 Pin12, J52 Pin14, J53 Pin16, J54 Pin18, J55 Pin20, J56 Pin22, J57 Pin24, J58 Pin26, J59 Pin28, J6 Pin9, J60 Pin30, J61 Pin32, J62 Pin34, J63 Pin36, J64 Pin38, J65 Pin40, J66 Pin42, J67 Pin44, J68 Pin46, J69 Pin48, J7 Pin11, J70 Pin50, J71 Pin52, J72 Pin54, J73 Pin56, J74 Pin58, J75 Pin60, J76 Pin62, J77 Pin64, J78 Pin66, J79 Pin68, J8 Pin13, J80 Pin70, J81 Pin72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

Commit message: Convert
Parts:
- G1: footprint rusefi_lib:LOGO -> gerefi_lib:LOGO
- G2: footprint rusefi_lib:Off_Road_Disclaimer -> gerefi_lib:Off_Road_Disclaimer
- J1: footprint rusefi_lib:BOSCH-88pin -> gerefi_lib:BOSCH-88pin
Other:
- board text added: "gerEFI - Bosch 88-pin Breakout R0.1"
- board text added: "https://github.com/gerefi/gerefi/tree/master/hardware"
- board text removed: "https://github.com/rusefi/rusefi/tree/master/hardware"
- board text removed: "rusEFI - Bosch 88-pin Breakout R0.1"
Changed lines of the file:
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@@
     (date 2020-06-03)
     (rev R0.1)
-    (company rusEFI)
+    (company gerEFI)
     (comment 1 Snake____1)
   )
@@
     )
   )
-  (module rusefi_lib:Off_Road_Disclaimer (layer F.Cu)
+  (module gerefi_lib:Off_Road_Disclaimer (layer F.Cu)
     (at 80.08 97.86 90)
     (fp_text reference G2 (at 0 -5.715 90) (layer F.SilkS) hide
@@
     )
   )
-  (module rusefi_lib:LOGO (layer F.Cu)
+  (module gerefi_lib:LOGO (layer F.Cu)
     (at 204.54 82.62)
     (fp_text reference G1 (at 0 4.14782) (layer F.SilkS) hide
@@
       (xy 3.3528 -0.39624)) (layer F.SilkS) (width 0.00254))
   )
-  (module rusefi_lib:BOSCH-88pin (layer F.Cu)
+  (module gerefi_lib:BOSCH-88pin (layer F.Cu)
     (at 146 123.5 180)
     (fp_text reference J1 (at 0 11.43) (layer F.SilkS)
@@
     (effects (font (size 1 1) (thickness 0.15)))
   )
-  (gr_text "rusEFI - Bosch 88-pin Breakout  R0.1" (at 215.97 96.59 270) (layer F.SilkS)
+  (gr_text "gerEFI - Bosch 88-pin Breakout  R0.1" (at 215.97 96.59 270) (layer F.SilkS)
     (effects (font (size 1 1) (thickness 0.15)))
   )
-  (gr_text https://github.com/rusefi/rusefi/tree/master/hardware (at 211 103 270) (layer F.SilkS)
+  (gr_text https://github.com/gerefi/gerefi/tree/master/hardware (at 211 103 270) (layer F.SilkS)
     (effects (font (size 1 1) (thickness 0.15)))
   )
