File: hardware/Breakout_Chip_TLE6244/Breakout_TLE6244.kicad_pcb (KiCad board)
At the start: 4 copper layers, 50.8 x 38.1 mm, 73 parts, among them K1 CONN_3, K2 CONN_3, K3 CONN_3, K4 CONN_3, K5 CONN_3, K6 CONN_3, K7 CONN_3, P1 CONN_4, P2 CONN_3, P3 CONN_2, P4 CONN_3, P5 CONN_5, P6 CONN_3, P7 CONN_2, P8 CONN_2, U1 TLE6244

Commit message: Convert
Other:
- board text added: "TLE6244 breakout R0.1 By DAECU for gerEFI"
- board text removed: "TLE6244 breakout R0.1 By DAECU for rusEFI"
Changed lines of the file:
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@@
     (title "Breakout TLE6244")
     (rev R.01)
-    (company http://rusefi.com/)
+    (company http://gerefi.com/)
   )
   (layers
@@
     (effects (font (size 0.508 0.508) (thickness 0.127)) (justify left mirror))
   )
-  (gr_text "TLE6244 breakout R0.1\nBy DAECU for rusEFI " (at 228.092 135.763) (layer B.SilkS)
+  (gr_text "TLE6244 breakout R0.1\nBy DAECU for gerEFI " (at 228.092 135.763) (layer B.SilkS)
     (effects (font (size 1.016 1.016) (thickness 0.254)) (justify mirror))
   )
