File: hardware/DDPAK_breakout/DDPAK_breakout.kicad_pcb (KiCad board)
At the start: 2 copper layers, 19.7 x 21.6 mm, 6 parts, among them P1 CONN_1, P2 CONN_2, P3 CONN_1, Q1 IRGS14C40L

Commit message: Convert
Other:
- board text added: "gerEFI by DAECU ignition R0.2 DDPAK breakout"
- board text removed: "rusEFI by DAECU ignition R0.2 DDPAK breakout"
Changed lines of the file:
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@@
     (title "DDPAK breakout")
     (rev R0.2)
-    (company rusEFI)
+    (company gerEFI)
   )
   (layers
@@
     (effects (font (size 0.889 0.889) (thickness 0.127)) (justify mirror))
   )
-  (gr_text "rusEFI by DAECU\nignition R0.2\nDDPAK breakout\n" (at 210.82 168.275 180) (layer B.SilkS)
+  (gr_text "gerEFI by DAECU\nignition R0.2\nDDPAK breakout\n" (at 210.82 168.275 180) (layer B.SilkS)
     (effects (font (size 0.889 0.889) (thickness 0.127)) (justify mirror))
   )
