File: hardware/DPAK2_breakout/DPAK2_breakout.kicad_pcb (KiCad board)
At the start: 2 copper layers, 16.5 x 19.1 mm, 6 parts, among them P1 CONN_1, P2 CONN_2, P3 CONN_1, Q1 IRGS14C40L

Commit message: Convert
Other:
- board text added: "gerEFI by DAECU ignition R0.1 DDPAK breakout"
- board text removed: "rusEFI by DAECU ignition R0.1 DDPAK breakout"
Changed lines of the file:
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@@
     (title "DDPAK breakout")
     (rev R0.1)
-    (company rusEFI)
+    (company gerEFI)
   )
   (layers
@@
     (effects (font (size 1.27 1.27) (thickness 0.127)) (justify mirror))
   )
-  (gr_text "rusEFI by DAECU\nignition R0.1\nDDPAK breakout\n" (at 209.804 168.402 90) (layer B.SilkS)
+  (gr_text "gerEFI by DAECU\nignition R0.1\nDDPAK breakout\n" (at 209.804 168.402 90) (layer B.SilkS)
     (effects (font (size 1.5 1.5) (thickness 0.3)) (justify mirror))
   )
