File: hardware/EEC-V-Blank-Board/eecv.kicad_pcb (KiCad board)
At the start: 2 copper layers, 140.8 x 164.4 mm, 1 part, among them J1 EEC-V

Commit message: Convert
Parts:
- J1: footprint rusefi_lib:eecv -> gerefi_lib:eecv
Changed lines of the file:
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@@
     (uvia_drill 0.1)
   )
-  (module rusefi_lib:eecv (layer F.Cu)
+  (module gerefi_lib:eecv (layer F.Cu)
     (at 93.63 20.44)
     (fp_text reference J1 (at 0 5.5) (layer F.SilkS)
