File: hardware/Power_regulator_TPS54340/TPS54340_Buck_Regulator.kicad_pcb (KiCad board)
At the start: 2 copper layers, 26 x 15.9 mm, 20 parts, among them J1 Conn_01x01, J2 Conn_01x01, J3 Conn_01x01, J4 Conn_01x01, J5 Conn_01x01, U1 TPS54340

Commit message: Convert
Other:
- board text added: "gerEFI.com"
- board text removed: "rusEFI.com"
Changed lines of the file:
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@@
     (date 2019-01-05)
     (rev R0.1)
-    (company "rusEFI by DAECU")
+    (company "gerEFI by DAECU")
   )
   (layers
@@
     (effects (font (size 2.032 1.524) (thickness 0.381)) (justify mirror))
   )
-  (gr_text rusEFI.com (at 181.61 125.095) (layer B.SilkS)
+  (gr_text gerEFI.com (at 181.61 125.095) (layer B.SilkS)
     (effects (font (size 2.032 1.524) (thickness 0.381)) (justify mirror))
   )
