File: hardware/TLF35584 breakout/TLF35584 breakout.kicad_pcb (KiCad board)
At the start: 2 copper layers, 70 x 35 mm, 41 parts, among them J1 POWER_IN, J2 SIGNALS, J3 POWER_IN, J4 POWER_OUT, Q1 DN2625K4, Q2 NTD2955T4G, Q3 NTD20N06LT4G, U1 TLF35584QKVS2

Commit message: Convert
Parts:
- G***: value rusEFI_logo_25mm -> gerEFI_logo_25mm; footprint TL35584 breakout:rusEFI_logo_25mm -> TL35584 breakout:gerEFI_logo_25mm
Changed lines of the file:
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@@
     )
   )
-  (module "TL35584 breakout:rusEFI_logo_25mm" (layer B.Cu)
+  (module "TL35584 breakout:gerEFI_logo_25mm" (layer B.Cu)
     (at 166.1 104.1 180)
     (fp_text reference G*** (at -0.05 7.4 180) (layer B.SilkS) hide
       (effects (font (size 1.524 1.524) (thickness 0.3)) (justify mirror))
     )
-    (fp_text value rusEFI_logo_25mm (at 0 -8 180) (layer B.SilkS) hide
+    (fp_text value gerEFI_logo_25mm (at 0 -8 180) (layer B.SilkS) hide
       (effects (font (size 1.524 1.524) (thickness 0.3)) (justify mirror))
     )
