File: hardware/VR_Board/vrs_io_1.kicad_pcb (KiCad board)
At the start: 2 copper layers, 38.1 x 12.7 mm, 38 parts, among them U101 MAX9926/9927

Commit message: Convert
Parts:
- G?: footprint rusEFI_lib:LOGO_F -> gerEFI_lib:LOGO_F
Other:
- board text added: "gerEFI.com"
- board text added: "gerEfi.com V 0.2"
- board text removed: "rusEFI.com"
- board text removed: "rusEfi.com V 0.2"
Changed lines of the file:
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@@
     (date 2018-12-15)
     (rev R0.2)
-    (company "rusEFI by DAECU")
+    (company "gerEFI by DAECU")
   )
   (layers
@@
       (net 17 /Cout2))
   )
-  (module rusEFI_lib:LOGO_F (layer B.Cu)
+  (module gerEFI_lib:LOGO_F (layer B.Cu)
     (at 212.725 121.92)
     (fp_text reference G? (at 0 -4.14782) (layer B.SilkS) hide
@@
   (gr_circle (center 189.865 125.73) (end 190.5 125.73) (layer Edge.Cuts) (width 0.254))
   (gr_circle (center 189.865 120.65) (end 190.5 120.65) (layer Edge.Cuts) (width 0.254))
-  (gr_text rusEFI.com (at 225.171 124.46 90) (layer F.SilkS)
+  (gr_text gerEFI.com (at 225.171 124.46 90) (layer F.SilkS)
     (effects (font (size 1 1) (thickness 0.127)))
   )
@@
   (gr_line (start 225.425 130.81) (end 205.105 130.81) (angle 90) (layer Edge.Cuts) (width 0.254))
   (gr_line (start 188.595 118.11) (end 225.425 118.11) (angle 90) (layer Edge.Cuts) (width 0.254))
-  (gr_text "rusEfi.com\n     V 0.2" (at 207.264 124.333 90) (layer B.SilkS)
+  (gr_text "gerEfi.com\n     V 0.2" (at 207.264 124.333 90) (layer B.SilkS)
     (effects (font (size 2.032 1.524) (thickness 0.381)) (justify mirror))
   )
