File: hardware/brain_board/brain_board_STM32F407.kicad_pcb (KiCad board)
At the start: 2 copper layers, 61.8 x 73.2 mm, 70 parts, among them J1 MINI-USB-5P-3400020P1, J2 MINI-USB-5P-3400020P1V, P1 CONN_25X2, P2 CONN_25X2, P3 CONN_2, P4 CONN_02X05, P5 CONN_01X03, P6 CONN_01X03, SW1 SW_PUSH, SW2 SW_PUSH, U1 STM32F407VG, U2 NUF2101MT1G, U3 LM2937, X1 CRYSTAL, X2 CRYSTAL(MC306)

Commit message: Convert
Parts:
- JP1, JP2, JP3, JP4: footprint rusEFI_LIB:SM0805_jumper -> gerEFI_LIB:SM0805_jumper
Other:
- board text added: "gerEFI.com R0.4"
- board text removed: "rusEFI.com R0.4"
Changed lines of the file:
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@@
     (date 2017-02-18)
     (rev R0.4)
-    (company "rusEFI by Art_Electro")
+    (company "gerEFI by Art_Electro")
   )
   (layers
@@
     )
   )
-  (module rusEFI_LIB:SM0805_jumper placed (layer F.Cu)
+  (module gerEFI_LIB:SM0805_jumper placed (layer F.Cu)
     (at 101.473 146.177 270)
     (attr smd)
@@
     )
   )
-  (module rusEFI_LIB:SM0805_jumper placed (layer F.Cu)
+  (module gerEFI_LIB:SM0805_jumper placed (layer F.Cu)
     (at 104.521 146.177 270)
     (attr smd)
@@
     )
   )
-  (module rusEFI_LIB:SM0805_jumper placed (layer F.Cu)
+  (module gerEFI_LIB:SM0805_jumper placed (layer F.Cu)
     (at 107.569 146.177 270)
     (attr smd)
@@
     )
   )
-  (module rusEFI_LIB:SM0805_jumper placed (layer F.Cu)
+  (module gerEFI_LIB:SM0805_jumper placed (layer F.Cu)
     (at 110.617 146.177 270)
     (attr smd)
@@
   )
   (gr_line (start 149.003 156.591) (end 87.217 156.591) (angle 90) (layer Edge.Cuts) (width 0.15))
-  (gr_text "rusEFI.com\nR0.4" (at 130.175 143.51) (layer F.SilkS)
+  (gr_text "gerEFI.com\nR0.4" (at 130.175 143.51) (layer F.SilkS)
     (effects (font (size 1.016 1.016) (thickness 0.2032)))
   )
