File: hardware/brain_board_176-pin/176-pin_board.kicad_pcb (KiCad board)
At the start: 4 copper layers, 61.8 x 73.2 mm, 77 parts, among them J1 MINI-USB-5P-3400020P1, P1 CONN_25X2, P10 CONN_2X2, P11 CONN_4X2, P12 CONN_4X2, P13 CONN_8X2, P2 CONN_25X2, P3 CONN_2, P4 CONN_6, P5 CONN_1, P6 CONN_2X2, P7 CONN_4X2, P8 CONN_4X2, P9 CONN_4X2, SW1 SW_PUSH, U1 STM32F407IGT6, U2 NUF2101MT1G, U3 LM2937, X1 CRYSTAL, X2 CRYSTAL(MC306)

Commit message: Convert
Other:
- board text added: "gerEfi.com STM32F4 176pin board ver 0.2"
- board text removed: "rusEfi.com STM32F4 176pin board ver 0.2"
Changed lines of the file:
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@@
     (title "176 pin board")
     (rev R0.2)
-    (company "rusEFI by Art_Electro & DAECU")
+    (company "gerEFI by Art_Electro & DAECU")
   )
   (layers
@@
     (pad 2 smd rect (at -15.485 0 90) (size 3.29 3.29) (layers B.Cu B.Paste B.Mask)
       (net 148 GND))
-    (model ../rusefi_lib/3d/MPD_CR2032.wrl
+    (model ../gerefi_lib/3d/MPD_CR2032.wrl
       (at (xyz 0 0 0))
       (scale (xyz 0.3937 0.3937 0.3937))
@@
     (pad 2 smd rect (at 1.04902 0 270) (size 1.19888 1.19888) (layers F.Cu F.Paste F.Mask)
       (net 148 GND))
-    (model ../rusefi_lib/3d/LED_0805.wrl
+    (model ../gerefi_lib/3d/LED_0805.wrl
       (at (xyz 0 0 0))
       (scale (xyz 1 1 1))
@@
     (pad "" thru_hole circle (at -2.159 -1.397 90) (size 1.016 1.016) (drill 0.762) (layers *.Cu *.Mask F.SilkS))
     (pad "" thru_hole circle (at 2.159 -1.397 90) (size 1.016 1.016) (drill 0.762) (layers *.Cu *.Mask F.SilkS))
-    (model ../rusefi_lib/3d/usb-2.wrl
+    (model ../gerefi_lib/3d/usb-2.wrl
       (at (xyz 0 0 0))
       (scale (xyz 1 1 1))
@@
     (pad 2 thru_hole rect (at -3.25 2.25 90) (size 2 1.5) (drill 1) (layers *.Cu *.Mask F.SilkS)
       (net 148 GND))
-    (model ../rusefi_lib/3d/pcb_push.wrl
+    (model ../gerefi_lib/3d/pcb_push.wrl
       (at (xyz 0 0 0))
       (scale (xyz 1 1 1))
@@
     (pad 2 smd rect (at 1.04902 0 270) (size 1.19888 1.19888) (layers F.Cu F.Paste F.Mask)
       (net 148 GND))
-    (model ../rusefi_lib/3d/LED_0805.wrl
+    (model ../gerefi_lib/3d/LED_0805.wrl
       (at (xyz 0 0 0))
       (scale (xyz 1 1 1))
@@
     (pad 2 smd rect (at 1.04902 0 270) (size 1.19888 1.19888) (layers F.Cu F.Paste F.Mask)
       (net 148 GND))
-    (model ../rusefi_lib/3d/LED_0805.wrl
+    (model ../gerefi_lib/3d/LED_0805.wrl
       (at (xyz 0 0 0))
       (scale (xyz 1 1 1))
@@
     (pad 2 smd rect (at 1.04902 0 270) (size 1.19888 1.19888) (layers F.Cu F.Paste F.Mask)
       (net 148 GND))
-    (model ../rusefi_lib/3d/LED_0805.wrl
+    (model ../gerefi_lib/3d/LED_0805.wrl
       (at (xyz 0 0 0))
       (scale (xyz 1 1 1))
@@
     (pad 2 smd rect (at 1.04902 0 270) (size 1.19888 1.19888) (layers F.Cu F.Paste F.Mask)
       (net 148 GND))
-    (model ../rusefi_lib/3d/LED_0805.wrl
+    (model ../gerefi_lib/3d/LED_0805.wrl
       (at (xyz 0 0 0))
       (scale (xyz 1 1 1))
@@
     (pad 2 smd rect (at 1.04902 0) (size 1.19888 1.19888) (layers F.Cu F.Paste F.Mask)
       (net 148 GND))
-    (model ../rusefi_lib/3d/LED_0805.wrl
+    (model ../gerefi_lib/3d/LED_0805.wrl
       (at (xyz 0 0 0))
       (scale (xyz 1 1 1))
@@
     (pad 2 smd rect (at 1.04902 0) (size 1.19888 1.19888) (layers F.Cu F.Paste F.Mask)
       (net 148 GND))
-    (model ../rusefi_lib/3d/LED_0805.wrl
+    (model ../gerefi_lib/3d/LED_0805.wrl
       (at (xyz 0 0 0))
       (scale (xyz 1 1 1))
@@
     (effects (font (size 0.762 0.762) (thickness 0.1524)))
   )
-  (gr_text "rusEfi.com STM32F4 176pin board ver 0.2" (at 116.84 149.86) (layer B.SilkS)
+  (gr_text "gerEfi.com STM32F4 176pin board ver 0.2" (at 116.84 149.86) (layer B.SilkS)
     (effects (font (size 1.016 1.016) (thickness 0.127)) (justify mirror))
   )
