File: hardware/brain_board_SD_Card_1/brain_board_SD_Card_1.kicad_pcb (KiCad board)
At the start: 2 copper layers, 14.6 x 33 mm, 6 parts, among them P352 MICRO-SDCARD-CONNECTOR-330006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, P5 CONN_01X03, P6 CONN_01X03

Commit message: Convert
Other:
- board text added: "gerEFI.com R0.1"
- board text removed: "rusEFI.com R0.1"
Changed lines of the file:
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@@
     (date 2016-12-31)
     (rev R0.1)
-    (company "rusEFI by DAECU")
+    (company "gerEFI by DAECU")
   )
   (layers
@@
     (pad "" thru_hole circle (at 3.407 -4.886) (size 0.889 0.889) (drill 0.762) (layers *.Cu *.Mask B.SilkS))
     (pad "" thru_hole circle (at 3.407 3.114) (size 0.889 0.889) (drill 0.762) (layers *.Cu *.Mask B.SilkS))
-    (model ../rusefi_lib/3d/9P-SMD-W-RING.wrl
+    (model ../gerefi_lib/3d/9P-SMD-W-RING.wrl
       (at (xyz -0.323 -0.33 -0.025))
       (scale (xyz 10 10 10))
@@
     )
   )
-  (gr_text "rusEFI.com\nR0.1" (at 179.07 129.667 270) (layer F.SilkS)
+  (gr_text "gerEFI.com\nR0.1" (at 179.07 129.667 270) (layer F.SilkS)
     (effects (font (size 1 1) (thickness 0.25)))
   )
