File: hardware/can_board/can_brd_1.kicad_pcb (KiCad board)
At the start: 2 copper layers, 32.1 x 10.9 mm, 13 parts, among them M471 CONN_1, P471 CONN_4, P472 CONN_2, P473 CONN_2, U471 SN65HVD230

Commit message: Convert
Other:
- board text added: "gerefi.com"
- board text removed: "rusefi.com"
Changed lines of the file:
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@@
       (net 6 GND)
     )
-    (model ../rusefi_lib/3d/LED_0805.wrl
+    (model ../gerefi_lib/3d/LED_0805.wrl
       (at (xyz 0 0 0))
       (scale (xyz 1 1 1))
@@
       (net 3 /CANL)
     )
-    (model ../rusefi_lib/3d/jumper-2.wrl
+    (model ../gerefi_lib/3d/jumper-2.wrl
       (at (xyz 0 0 0))
       (scale (xyz 1 1 1))
@@
     (effects (font (size 0.762 0.762) (thickness 0.1016)) (justify mirror))
   )
-  (gr_text rusefi.com (at 152.654 184.2516) (layer B.SilkS)
+  (gr_text gerefi.com (at 152.654 184.2516) (layer B.SilkS)
     (effects (font (size 0.762 0.762) (thickness 0.075)) (justify mirror))
   )
