File: hardware/hip9011/DD_HIP9011.kicad_pcb (KiCad board)
At the start: 2 copper layers, 40 x 34 mm, 37 parts, among them P161 KNOCK 1, P162 KNOCK 2, P163 12V, P164 CONN_5X2, P165 CONN_2, P166 CONN_2, U131 7805-SOT89, X161 CRYSTAL

Commit message: Convert
Other:
- board text added: "DD_HIP9011 Rev.1 www.gerefi.com"
- board text removed: "DD_HIP9011 Rev.1 www.rusefi.com"
Changed lines of the file:
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@@
     (arrow2b (pts (xy 113.999999 21) (xy 114.586419 22.126503)))
   )
-  (gr_text "DD_HIP9011 Rev.1\nwww.rusefi.com\n" (at 94.234 25.781) (layer B.SilkS)
+  (gr_text "DD_HIP9011 Rev.1\nwww.gerefi.com\n" (at 94.234 25.781) (layer B.SilkS)
     (effects (font (size 1.5 1.5) (thickness 0.3)) (justify left mirror))
   )
