File: hardware/low_side_tle6240/tle6240_driver.kicad_pcb (KiCad board)
At the start: 2 copper layers, 42.7 x 56.5 mm, 12 parts, among them K1 JUMPER3, K2 CONN_3, P1 CONN_10X2, P2 CONN_16, P3 CONN_2X2

Commit message: Convert
Other:
- board text added: "for gerEFI rev 00.11"
- board text removed: "for rusEFI rev 00.11"
Changed lines of the file:
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@@
   (page A)
   (title_block
-    (title "rusEFI break out board")
+    (title "gerEFI break out board")
     (date 2018-12-29)
     (rev R0.1)
@@
     (arrow2b (pts (xy 175.768 153.161999) (xy 176.894504 152.575578)))
   )
-  (gr_text "for rusEFI\nrev 00.11" (at 198.12 116.84) (layer F.SilkS)
+  (gr_text "for gerEFI\nrev 00.11" (at 198.12 116.84) (layer F.SilkS)
     (effects (font (size 1.5 1.5) (thickness 0.3)))
   )
