File: hardware/usb_mmc_spi/mmc_usb_1.kicad_pcb (KiCad board)
At the start: 2 copper layers, 47.6 x 27.3 mm, 27 parts, among them J351 MINI-USB-5P-3400020P1, K351 CONN_3, M351 CONN_1, M352 CONN_1, P351 CONN_5X2, P352 MICRO-SDCARD-CONNECTOR-330006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, P353 CONN_10X2, P354 CONN_10X2, P355 CONN_1, P356 CONN_1, U351 FT232RL

Commit message: Convert
Other:
- board text added: "gerEfi.com USB+SD ver 0.3"
- board text removed: "rusEfi.com USB+SD ver 0.3"
Changed lines of the file:
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@@
       (net 16 GND)
     )
-    (model ../rusefi_lib/3d/LED_0805.wrl
+    (model ../gerefi_lib/3d/LED_0805.wrl
       (at (xyz 0 0 0))
       (scale (xyz 1 1 1))
@@
       (net 16 GND)
     )
-    (model ../rusefi_lib/3d/LED_0805.wrl
+    (model ../gerefi_lib/3d/LED_0805.wrl
       (at (xyz 0 0 0))
       (scale (xyz 1 1 1))
@@
       (net 16 GND)
     )
-    (model ../rusefi_lib/3d/LED_0805.wrl
+    (model ../gerefi_lib/3d/LED_0805.wrl
       (at (xyz 0 0 0))
       (scale (xyz 1 1 1))
@@
       (layers *.Cu *.Mask F.SilkS)
     )
-    (model ../rusefi_lib/3d/usb-2.wrl
+    (model ../gerefi_lib/3d/usb-2.wrl
       (at (xyz 0 0 0))
       (scale (xyz 1 1 1))
@@
       (layers *.Cu *.Mask F.SilkS)
     )
-    (model ../rusefi_lib/3d/9P-SMD-W-RING.wrl
+    (model ../gerefi_lib/3d/9P-SMD-W-RING.wrl
       (at (xyz -0.323 -0.33 -0.025))
       (scale (xyz 10 10 10))
@@
       (net 7 /CS4)
     )
-    (model ../rusefi_lib/3d/M_header_5x2.wrl
+    (model ../gerefi_lib/3d/M_header_5x2.wrl
       (at (xyz 0 0 0))
       (scale (xyz 1 1 1))
@@
       (net 37 N-0000037)
     )
-    (model ../rusefi_lib/3d/M_header_10x2.wrl
+    (model ../gerefi_lib/3d/M_header_10x2.wrl
       (at (xyz 0 0 0))
       (scale (xyz 1 1 1))
@@
       (net 16 GND)
     )
-    (model ../rusefi_lib/3d/M_header_10x2.wrl
+    (model ../gerefi_lib/3d/M_header_10x2.wrl
       (at (xyz 0 0 0))
       (scale (xyz 1 1 1))
@@
   (gr_line (start 127 187.96) (end 129.54 187.96) (angle 90) (layer Cmts.User) (width 0.2))
   (gr_line (start 127 127) (end 127 187.96) (angle 90) (layer Cmts.User) (width 0.2))
-  (gr_text "rusEfi.com USB+SD ver 0.3" (at 198.628 160.401) (layer B.SilkS)
+  (gr_text "gerEfi.com USB+SD ver 0.3" (at 198.628 160.401) (layer B.SilkS)
     (effects (font (size 1 1) (thickness 0.25)) (justify mirror))
   )
